Commit message: update the model of gripper

File: robots/z1_description/xacro/robot.xacro (robot description, xacro)
@@ -289,6 +289,6 @@
         <link name="realsense_mountpoint"/>
         <joint name="realsense_mountpoint_joint" type="fixed">
-            <origin xyz="0.148 0 0.084" rpy="0 0.175 0" />
-            <parent link="link06"/>
+            <origin xyz="-0.043 0 0.07" rpy="0 0.1745 0" />
+            <parent link="link_gripper"/>
             <child link="realsense_mountpoint" />
         </joint>
@@ -297,5 +297,5 @@
     <xacro:if value="$(arg HitbotGripper)">
         <joint name="gripper_mount" type="fixed">
-            <origin xyz="0.1 0 -0.08" rpy="0 0 0" />
+            <origin xyz="0.0513 0 0" rpy="0 0 0" />
             <parent link="link06"/>
             <child link="link_gripper" />
@@ -316,5 +316,5 @@
                 <origin xyz="0 0 0" rpy="0 0 0" />
                 <geometry>
-                    <mesh filename="package://z1_description/meshes/visual/hitbot_gripper.STL" />
+                    <mesh filename="package://z1_description/meshes/visual/gripper_body.dae" />
                 </geometry>
                 <material name="">
@@ -325,5 +325,83 @@
                 <origin xyz="0 0 0" rpy="0 0 0" />
                 <geometry>
-                    <mesh filename="package://z1_description/meshes/visual/hitbot_gripper.STL" />
+                    <mesh filename="package://z1_description/meshes/visual/gripper_body.dae" />
+                </geometry>
+            </collision>
+        </link>
+        <joint name="gripper_1" type="fixed">
+            <origin xyz="0.087 0 -0.0005" rpy="0 0 0" />
+            <parent link="link_gripper"/>
+            <child link="link_gripper_1" />
+            <axis xyz="0 1 0" />
+            <limit
+                lower="0"
+                upper="0.2"
+                effort="2000"
+                velocity="1" />
+        </joint>
+        <link name="link_gripper_1">
+            <inertial>
+                <origin xyz="0 0 0" rpy="0 0 0" />
+                <mass value="0.290087803254386" />
+                <inertia
+                    ixx="0.000122722161885507"
+                    ixy="2.8456952860616E-06"
+                    ixz="3.69598304197937E-06"
+                    iyy="0.000255921213582023"
+                    iyz="1.99093327058819E-07"
+                    izz="0.00032692475873505" />
+                </inertial>
+            <visual>
+                <origin xyz="0 0 0" rpy="0 0 0" />
+                <geometry>
+                    <mesh filename="package://z1_description/meshes/visual/gripper_1.dae" />
+                </geometry>
+                <material name="">
+                    <color  rgba="0.792156862745098 0.819607843137255 0.933333333333333 1" />
+                </material>
+            </visual>
+            <collision>
+                <origin xyz="0 0 0" rpy="0 0 0" />
+                <geometry>
+                    <mesh filename="package://z1_description/meshes/visual/gripper_1.dae" />
+                </geometry>
+            </collision>
+        </link>
+        <joint name="gripper_2" type="fixed">
+            <origin xyz="0.087 0 -0.0005" rpy="0 0 0" />
+            <parent link="link_gripper"/>
+            <child link="link_gripper_2" />
+            <axis xyz="0 -1 0" />
+            <limit
+                lower="0"
+                upper="0.2"
+                effort="2000"
+                velocity="1" />
+        </joint>
+        <link name="link_gripper_2">
+            <inertial>
+                <origin xyz="0 0 0" rpy="0 0 0" />
+                <mass value="0.290087803254386" />
+                <inertia
+                    ixx="0.000122722161885507"
+                    ixy="2.8456952860616E-06"
+                    ixz="3.69598304197937E-06"
+                    iyy="0.000255921213582023"
+                    iyz="1.99093327058819E-07"
+                    izz="0.00032692475873505" />
+                </inertial>
+            <visual>
+                <origin xyz="0 0 0" rpy="0 0 0" />
+                <geometry>
+                    <mesh filename="package://z1_description/meshes/visual/gripper_2.dae" />
+                </geometry>
+                <material name="">
+                    <color  rgba="0.792156862745098 0.819607843137255 0.933333333333333 1" />
+                </material>
+            </visual>
+            <collision>
+                <origin xyz="0 0 0" rpy="0 0 0" />
+                <geometry>
+                    <mesh filename="package://z1_description/meshes/visual/gripper_2.dae" />
                 </geometry>
             </collision>

Commit message: modified some parameters

File: robots/z1_description/xacro/robot.xacro (robot description, xacro)
@@ -289,6 +289,6 @@
         <link name="realsense_mountpoint"/>
         <joint name="realsense_mountpoint_joint" type="fixed">
-            <origin xyz="-0.043 0 0.07" rpy="0 0.1745 0" />
-            <parent link="link_gripper"/>
+            <origin xyz="0.01 0 0.07" rpy="0 0.1745 0" />
+            <parent link="link06"/>
             <child link="realsense_mountpoint" />
         </joint>
@@ -297,5 +297,5 @@
     <xacro:if value="$(arg HitbotGripper)">
         <joint name="gripper_mount" type="fixed">
-            <origin xyz="0.0513 0 0" rpy="0 0 0" />
+            <origin xyz="0.0514 0 0" rpy="0 0 0" />
             <parent link="link06"/>
             <child link="link_gripper" />
@@ -330,13 +330,13 @@
         </link>
         <joint name="gripper_1" type="fixed">
-            <origin xyz="0.087 0 -0.0005" rpy="0 0 0" />
+            <origin xyz="0.097 0 -0.0005" rpy="0 0 0" />
             <parent link="link_gripper"/>
             <child link="link_gripper_1" />
-            <axis xyz="0 1 0" />
+            <!-- <axis xyz="0 1 0" />
             <limit
                 lower="0"
                 upper="0.2"
                 effort="2000"
-                velocity="1" />
+                velocity="1" /> -->
         </joint>
         <link name="link_gripper_1">
@@ -369,5 +369,5 @@
         </link>
         <joint name="gripper_2" type="fixed">
-            <origin xyz="0.087 0 -0.0005" rpy="0 0 0" />
+            <origin xyz="0.097 0 -0.0005" rpy="0 0 0" />
             <parent link="link_gripper"/>
             <child link="link_gripper_2" />
